File: modules/UPModule/SB_TS_2.00.brd (EAGLE design)
At the start: 42.3 x 27.4 mm, 67 parts, among them IC1 MC34063AD, IC2 MCP1702-33, IC3 LPC922FDH, Q1 BC856, Q2 BCP52, T1 BC848, T2 BC848

Commit message: update produktions stand.
Parts:
- moved R2 5.17 mm to (12.4, 25.5)
Routing:
- net PWM: track 40.7 -> 35.9 mm
- net VCC: track 74.3 -> 71.7 mm
- net N$6: track 0.00 -> 1.98 mm, vias 1 -> 0
- net TXD: track 51.3 -> 50.5 mm
- net N$19: track 6.35 -> 6.85 mm
- net GND: vias 11 -> 22
